File: MiniBee.kicad_pcb (KiCad board)
At the start: 2 copper layers, 23.2 x 22 mm, 40 parts, among them J1 USB, J4 SK6812, P1 TC2030-CTX-Tag-Connect, SW1 DFU, U1 USBLC4SC6, U2 STM32WB5MMG, U3 SY8201

Commit message: updated project files
Connections:
- U2 pad 28: T3 -> unconnected-(U2-Pad28)
- U2 pad 51: T2 -> unconnected-(U2-Pad51)
- U2 pad 52: unconnected-(U2-Pad52) -> T1
Routing:
- net T1: track 5.45 -> 6.78 mm
Other:
- board text added: "MiniBee 2023 v1.1.0"
- board text removed: "MiniBee 2023 v1.0.0"
